File: R1/RAMA_M10-A_R1.brd (EAGLE design)
At the start: 80 x 100 mm, 40 parts, among them Q2 PCHANNEL-MOSFET, Y1 16MHz

Commit message: Rounded corners, strengthened mounting holes, changed fonts to nicer hand-drawn font, altered USB & TQFN-44 footprints, fixed incorrectly reversed MISO/MOSI, altered copper pour on RAMA & Machine logos
Connections:
- net MISO: now also U$8.11; no longer U$8.10
- net MOSI: now also U$8.10; no longer U$8.11
Routing:
- net N$32: track 22.8 -> 0.00 mm
- net N$28: track 6.06 -> 0.00 mm
- net N$31: track 5.83 -> 0.00 mm
- net N$30: track 5.41 -> 0.00 mm
- net N$29: track 5.41 -> 0.00 mm
- net SCK: track 19.6 -> 21.3 mm
- net VCC: track 173.2 -> 174.7 mm
- net MISO: track 22.9 -> 23.5 mm
Other:
- outline, holes or cut-outs redrawn
- board text removed: "10 KEY PROGRAMMABLE KEYPAD"
- board text removed: "5V PLANE"
- board text removed: "ASSEMBLED IN THE UK"
- board text removed: "BOARD MODEL"
- board text removed: "CAUTION: MAXIMUM VOLTAGE 5.2V"
- board text removed: "CHECKED BY:"
- board text removed: "GND"
- board text removed: "GND PLANE"
- board text removed: "Github.com/MachineIndustries/M10-A"
- board text removed: "IN COLLABORATION WITH RAMAWORKS"
- board text removed: "ISSUE NO:"
- board text removed: "M10-A"
- board text removed: "M10-A-R1 / MIN-7R1"
- board text removed: "MACHINEINDUSTRIES.CO"
- board text removed: "MISO"
- board text removed: "MOSI"
- board text removed: "OPEN SOURCE HARDWARE"
- board text removed: "POS-A"
- board text removed: "POS-B"
- board text removed: "POS-C"
- board text removed: "POS-D"
- board text removed: "PROTOTYPE"
- board text removed: "R1"
- board text removed: "RAMA + MACHINE INDUSTRIES"
- board text removed: "RESET"
- board text removed: "RST"
- board text removed: "SCK"
- board text removed: "SERIAL NO. MIN-7R1P1"
- board text removed: "VCC"

Commit message: Pre-prod
Parts:
- removed R4: 1k, Adafruit Bluefruit LE nRF8001:_0603MP
- added ISP2: AVRISP-SMT, adafruit:AVRISP-SMT
- added JP1: (no value), SparkFun-Connectors:1X06
- added R10, R11, R12, R13, R14, R15, R16, R7, R8, R9: 100ohm, Adafruit Bluefruit LE nRF8001:_0603MP
- added R6: 10k, Adafruit Bluefruit LE nRF8001:_0603MP
- moved TP2 6.48 mm to (26.9, 19.0)
- moved Q2 1.61 mm to (29.4, 18.5), turned to 180 degrees
- moved C3 0.50 mm to (22.8, 30.4)
- moved C6 0.50 mm to (14.8, 30.4)
- moved R3 0.50 mm to (13.1, 30.4)
Connections:
- removed net N$4: Q2.2, R4.2
- new net JP_GND: ISP2.6, JP1.6
- new net JP_MISO: ISP2.1, JP1.1
- new net JP_RST: ISP2.5, JP1.3
- new net JP_SCK: ISP2.3, JP1.2
- new net JP_VCC: ISP2.2, JP1.4
- new net N$28: KEY7.LED2, R13.2
- new net N$29: KEY8.LED2, R14.2
- new net N$30: KEY9.LED2, R15.2
- new net N$31: KEY10.LED2, R16.2
- new net N$32: KEY4.LED2, R10.2
- new net N$69: KEY5.LED2, R11.2
- new net N$70: KEY6.LED2, R12.2
- new net N$71: KEY3.LED2, R9.2
- new net N$72: KEY2.LED2, R8.2
- new net N$73: KEY1.LED2, R7.2
- new net N$74: ISP2.4, JP1.5
- net 5V: now also Q2.3; no longer R4.1
- net GND: now also R10.1, R11.1, R12.1, R13.1, R14.1, R15.1, R16.1, R7.1, R8.1, R9.1; no longer KEY1.LED2, KEY10.LED2, KEY2.LED2, KEY3.LED2, KEY4.LED2, KEY5.LED2, KEY6.LED2, KEY7.LED2, KEY8.LED2, KEY9.LED2
- net N$13: now also R6.2
- net VCC: now also Q2.2, R6.1; no longer Q2.3
Routing:
- net N$74: track 0.00 -> 15.9 mm, vias 0 -> 2
- net JP_VCC: track 0.00 -> 13.8 mm, vias 0 -> 1
- net JP_GND: track 0.00 -> 13.6 mm, vias 0 -> 1
- net JP_MISO: track 0.00 -> 9.13 mm
- net JP_SCK: track 0.00 -> 9.13 mm
- net JP_RST: track 0.00 -> 9.13 mm
- net COL2: track 91.3 -> 86.0 mm
- net VCC: track 174.7 -> 178.0 mm
- net N$31: track 0.00 -> 3.08 mm
- net N$73: track 0.00 -> 2.97 mm
- net N$72: track 0.00 -> 2.97 mm
- net N$71: track 0.00 -> 2.97 mm
- net N$70: track 0.00 -> 2.97 mm
- net N$69: track 0.00 -> 2.97 mm
- net N$32: track 0.00 -> 2.97 mm
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Other:
- board size 80 x 100 mm -> 99 x 100 mm
